Commit message: force fetch with randomized ball pos

File: robots/simplified_fetch.urdf (robot description, URDF)
Before this commit: robot fetch, 11 links, 10 joints
Links:
- added link force_link_front, mass 0; collision box size=0.05 0.5 0.05; visual box size=0.05 0.5 0.05
Joints:
- added joint force_front_joint: type fixed, parent base_link, child force_link_front, origin xyz=0.3 0 0.1 rpy=0 0 0, axis 0 1 0
